Commit message: Actualiza URDF y colisiones del robot

File: src/lak_description/urdf/lak_obedience.urdf (robot description, URDF)
Before this commit: robot lak_obedience_robot, 23 links, 22 joints
Links:
- link body_assembly_1: geometry collision box size=0.19 0.10 0.14; visual mesh filename=package://lak_description/meshes/visual/body_assembly_1.stl
- link foot_assembly_1: geometry collision box size=0.1 0.03 0.045; visual mesh filename=package://lak_description/meshes/visual/foot_assembly_1.stl
- link foot_assembly_2: geometry collision box size=0.1 0.03 0.045; visual mesh filename=package://lak_description/meshes/visual/foot_assembly_2.stl
- link head_assembly_1: geometry collision box size=0.05 0.15 0.20; visual mesh filename=package://lak_description/meshes/visual/head_assembly_1.stl
- link left_cache_1: geometry collision box size=0.08 0.16 0.03; visual mesh filename=package://lak_description/meshes/visual/left_cache_1.stl
- link right_cache_1: geometry collision box size=0.08 0.16 0.03; visual mesh filename=package://lak_description/meshes/visual/right_cache_1.stl
- link trunk_assembly_1: geometry visual mesh filename=package://lak_description/meshes/visual/trunk_assembly_1.stl
Joints:
- joint chasis_joint: origin xyz=0 0 0.1 rpy=0 0 0 -> xyz=0 0 0.174 rpy=0 0 0
- joint dof_head_pitch: limit lower=-6.2831853 upper=6.2831853 effort=1 velocity=1 -> lower=-0.785398 upper=0.785398 effort=1 velocity=1
- joint dof_head_roll: limit lower=-6.2831853 upper=6.2831853 effort=1 velocity=1 -> lower=-0.523599 upper=0.523599 effort=1 velocity=1
- joint dof_head_yaw: limit lower=-6.2831853 upper=6.2831853 effort=1 velocity=1 -> lower=-2.96706 upper=2.96706 effort=1 velocity=1
- joint dof_left_ankle: limit lower=-6.2831853 upper=6.2831853 effort=1 velocity=1 -> lower=-1.5708 upper=1.5708 effort=1 velocity=1
- joint dof_left_hip_pitch: limit lower=-6.2831853 upper=6.2831853 effort=1 velocity=1 -> lower=-1.22173 upper=0.523599 effort=1 velocity=1
- joint dof_left_hip_roll: limit lower=-6.2831853 upper=6.2831853 effort=1 velocity=1 -> lower=-0.436332 upper=0.436332 effort=1 velocity=1
- joint dof_left_hip_yaw: limit lower=-6.2831853 upper=6.2831853 effort=1 velocity=1 -> lower=-0.523599 upper=0.523599 effort=1 velocity=1; origin xyz=-0.081685897 0.036856802 0.15174282 rpy=1.5509545e-16 0 0 -> xyz=0.01 0.036856802 0.0698310383 rpy=1.5509545e-16 0 0
- joint dof_left_knee: limit lower=-6.2831853 upper=6.2831853 effort=1 velocity=1 -> lower=-1.5708 upper=1.5708 effort=1 velocity=1
- joint dof_neck_pitch: limit lower=-6.2831853 upper=6.2831853 effort=1 velocity=1 -> lower=-0.349066 upper=1.13446 effort=1 velocity=1; origin xyz=-0.061685897 0.021006802 0.19580282 rpy=1.5707963 0 -3.3306691e-16 -> xyz=0.03 0.021006802 0.1138910383 rpy=1.5707963 0 -3.3306691e-16
- joint dof_right_ankle: limit lower=-6.2831853 upper=6.2831853 effort=1 velocity=1 -> lower=-1.5708 upper=1.5708 effort=1 velocity=1
- joint dof_right_hip_pitch: limit lower=-6.2831853 upper=6.2831853 effort=1 velocity=1 -> lower=-0.523599 upper=1.22173 effort=1 velocity=1
- joint dof_right_hip_roll: limit lower=-6.2831853 upper=6.2831853 effort=1 velocity=1 -> lower=-0.436332 upper=0.436332 effort=1 velocity=1
- joint dof_right_hip_yaw: limit lower=-6.2831853 upper=6.2831853 effort=1 velocity=1 -> lower=-0.523599 upper=0.523599 effort=1 velocity=1; origin xyz=-0.081685897 -0.033143198 0.15174282 rpy=-1.5509545e-16 0 0 -> xyz=0.01 -0.033143198 0.0698310383 rpy=-1.5509545e-16 0 0
- joint dof_right_knee: limit lower=-6.2831853 upper=6.2831853 effort=1 velocity=1 -> lower=-1.5708 upper=1.5708 effort=1 velocity=1
- joint fix_body_bottom: origin xyz=-0.091685897 0.011856802 0.081917817 rpy=0 0 0 -> xyz=0.0 0.011856802 0.0 rpy=0 0 0
- joint fix_left_antenna: limit lower=-6.2831853 upper=6.2831853 effort=1 velocity=1 -> lower=-1.5708 upper=1.5708 effort=1 velocity=1
- joint fix_right_antenna: limit lower=-6.2831853 upper=6.2831853 effort=1 velocity=1 -> lower=-1.5708 upper=1.5708 effort=1 velocity=1

Commit message: Update URDF Files for Pybullet

File: src/lak_description/urdf/lak_obedience.urdf (robot description, URDF)
Before this commit: robot lak_obedience_robot, 23 links, 22 joints
Links:
- removed link base_link
- removed link trunk_assembly_1
- added link trunk_link, mass 0.30884485; collision mesh filename=package://lak_description/meshes/collision/trunk_assembly_1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; visual mesh filename=package://lak_description/meshes/collision/trunk_assembly_1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
- link antenna_1: geometry collision mesh filename=package://lak_description/meshes/collision/antenna_1.stl; visual mesh filename=package://lak_description/meshes/collision/antenna_1.stl
- link antenna_2: geometry collision mesh filename=package://lak_description/meshes/collision/antenna_2.stl; visual mesh filename=package://lak_description/meshes/collision/antenna_2.stl
- link body_assembly_1: geometry collision mesh filename=package://lak_description/meshes/collision/body_assembly_1.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; visual mesh filename=package://lak_description/meshes/collision/body_assembly_1.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
- link foot_assembly_1: geometry collision mesh filename=package://lak_description/meshes/collision/foot_assembly_1.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; visual mesh filename=package://lak_description/meshes/collision/foot_assembly_1.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
- link foot_assembly_2: geometry collision mesh filename=package://lak_description/meshes/collision/foot_assembly_2.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; visual mesh filename=package://lak_description/meshes/collision/foot_assembly_2.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
- link head_assembly_1: geometry collision mesh filename=package://lak_description/meshes/collision/head_assembly_1.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; visual mesh filename=package://lak_description/meshes/collision/head_assembly_1.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
- link head_pitch_to_yaw_1: geometry collision mesh filename=package://lak_description/meshes/collision/head_pitch_to_ya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; visual mesh filename=package://lak_description/meshes/collision/head_pitch_to_ya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
- link hip_roll_assembly_1: geometry collision mesh filename=package://lak_description/meshes/collision/hip_roll_assembl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; visual mesh filename=package://lak_description/meshes/collision/hip_roll_assembl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
- link hip_roll_assembly_2: geometry collision mesh filename=package://lak_description/meshes/collision/hip_roll_assembl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; visual mesh filename=package://lak_description/meshes/collision/hip_roll_assembl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
- link knee_and_ankle_assembly_1: geometry collision mesh filename=package://lak_description/meshes/collision/knee_and_ankle_a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; visual mesh filename=package://lak_description/meshes/collision/knee_and_ankle_a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
- link knee_and_ankle_assembly_2: geometry collision mesh filename=package://lak_description/meshes/collision/knee_and_ankle_a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; visual mesh filename=package://lak_description/meshes/collision/knee_and_ankle_a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
- link knee_and_ankle_assembly_3: geometry collision mesh filename=package://lak_description/meshes/collision/knee_and_ankle_a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; visual mesh filename=package://lak_description/meshes/collision/knee_and_ankle_a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
- link knee_and_ankle_assembly_4: geometry collision mesh filename=package://lak_description/meshes/collision/knee_and_ankle_a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; visual mesh filename=package://lak_description/meshes/collision/knee_and_ankle_a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
- link left_antenna_holder_1: geometry collision mesh filename=package://lak_description/meshes/collision/left_antenna_hol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; visual mesh filename=package://lak_description/meshes/collision/left_antenna_hol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
- link left_cache_1: geometry collision mesh filename=package://lak_description/meshes/collision/left_cache_1.stl; visual mesh filename=package://lak_description/meshes/collision/left_cache_1.stl
- link left_roll_to_pitch_assembly_1: geometry collision mesh filename=package://lak_description/meshes/collision/left_roll_to_pit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; visual mesh filename=package://lak_description/meshes/collision/left_roll_to_pit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
- link neck_pitch_assembly_1: geometry collision mesh filename=package://lak_description/meshes/collision/neck_pitch_assem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; visual mesh filename=package://lak_description/meshes/collision/neck_pitch_assem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
- link neck_yaw_assembly_1: geometry collision mesh filename=package://lak_description/meshes/collision/neck_yaw_assembl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; visual mesh filename=package://lak_description/meshes/collision/neck_yaw_assembl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
- link right_antenna_holder_1: geometry collision mesh filename=package://lak_description/meshes/collision/right_antenna_ho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; visual mesh filename=package://lak_description/meshes/collision/right_antenna_ho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
- link right_cache_1: geometry collision mesh filename=package://lak_description/meshes/collision/right_cache_1.stl; visual mesh filename=package://lak_description/meshes/collision/right_cache_1.stl
- link right_roll_to_pitch_assembly_1: geometry collision mesh filename=package://lak_description/meshes/collision/right_roll_to_pi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; visual mesh filename=package://lak_description/meshes/collision/right_roll_to_pi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
Joints:
- removed joint chasis_joint
- joint dof_left_hip_yaw: parent trunk_assembly_1 -> trunk_link
- joint dof_neck_pitch: parent trunk_assembly_1 -> trunk_link
- joint dof_right_hip_yaw: parent trunk_assembly_1 -> trunk_link
- joint fix_body_bottom: parent trunk_assembly_1 -> trunk_link
- joint fix_left_antenna: type revolute -> fixed
- joint fix_right_antenna: type revolute -> fixed

File: src/lak_description/urdf/lak_obedience_v2.urdf (robot description, URDF)
Before this commit: robot lak-obedience, 20 links, 19 joints
Links:
- link L_hip_yaw_link: geometry collision mesh filename=package://lak_description/meshes_v2/collision/drive_palonie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; collision mesh filename=package://lak_description/meshes_v2/collision/passive_palon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
- link base_link: geometry collision mesh filename=package://lak_description/meshes_v2/collision/acrilico.stl; collision mesh filename=package://lak_description/meshes_v2/collision/battery_pack_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
- link head_link: geometry collision mesh filename=package://lak_description/meshes_v2/collision/antenna.stl; collision mesh filename=package://lak_description/meshes_v2/collision/antenna.stl
